Commit message: Setup for LiDAR

File: src/ackermann_vehicle_description/urdf/lidar.xacro (robot description, xacro)
@@ -3,8 +3,8 @@
     <joint name="head_lidar_joint" type="fixed">
         <parent link="base_link"/>
-        <child link="head_lidar"/>
+        <child link="horizontal_laser_link"/>
         <origin xyz="0 0 0.1" rpy="0 0 0"/>
     </joint>
-    <link name="head_lidar">
+    <link name="horizontal_laser_link">
         <visual>
             <geometry>
@@ -14,10 +14,10 @@
         </visual>
     </link>
-    <gazebo reference="head_lidar">
+    <gazebo reference="horizontal_laser_link">
         <material>Gazebo/Red</material>
         <sensor name="head_lidar_sensor" type="ray">
             <pose> 0 0 0 0 0 0 </pose>
-            <visualize>false</visualize>
-            <update_rate>40</update_rate>
+            <visualize>true</visualize>
+            <update_rate>10</update_rate>
             <ray>
                 <scan>
@@ -30,6 +30,6 @@
                 </scan>
                 <range>
-                    <min>0.1</min>
-                    <max>10.0</max>
+                    <min>0.15</min>
+                    <max>12.0</max>
                 </range>
                 <noise>
@@ -44,6 +44,6 @@
             </ray>
             <plugin name="laser_controller" filename="libgazebo_ros_laser.so">
-                <topicName>laser/scan</topicName>
-                <frameName>head_lidar</frameName>
+                <topicName>/scan</topicName>
+                <frameName>horizontal_laser_link</frameName>
             </plugin>
         </sensor>

File: src/ackermann_vehicle_description/urdf/rc_car.xacro (robot description, xacro)
@@ -2,7 +2,8 @@
 <robot xmlns:xacro="http://www.ros.org/wiki/xacro"  name="soonduck">
     <xacro:include filename="body.xacro" />
-    <!-- <xacro:include filename="lidar.xacro"/> -->
+    <xacro:include filename="lidar.xacro"/>
     <!-- <xacro:include filename="lidar_3d.xacro"/> -->
-    <xacro:include filename="ir.xacro"/>
+    <!-- <xacro:include filename="ir.xacro"/> -->
     <!-- <xacro:include filename="camera.xacro"/> -->
+    <xacro:include filename="imu.xacro"/>
 </robot>
